File: sweepish/sweepish.kicad_pcb (KiCad board)
At the start: 2 copper layers, 117 x 91.4 mm, 35 parts, among them U1 XIAO-nRF52840-DIP

Commit message: Uploaded KiCad Files
Connections:
- U1 pad 6: Col 4 -> Col 3
- U1 pad 7: Col 3 -> Col 4
Routing:
- net Col 3: track 107.7 -> 98.4 mm
- net Col 4: track 99.2 -> 92.8 mm
- added copper zone on B.Cu, net Col 4
- added copper zone on F.Cu, net Col 4
- removed copper zone on B.Cu, net (none)
- removed copper zone on F.Cu, net (none)
Changed lines of the file:
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@@
 			(layers "F.Cu" "F.Mask")
 			(roundrect_rratio 0.1)
-			(net 26 "Col 4")
+			(net 25 "Col 3")
 			(pinfunction "P0.05_AIN3_A5_D5")
 			(pintype "passive")
@@
 			(layers "*.Cu" "*.Mask")
 			(remove_unused_layers no)
-			(net 26 "Col 4")
+			(net 25 "Col 3")
 			(pinfunction "P0.05_AIN3_A5_D5")
 			(pintype "passive")
@@
 			(layers "F.Cu" "F.Mask")
 			(roundrect_rratio 0.1)
-			(net 25 "Col 3")
+			(net 26 "Col 4")
 			(pinfunction "P1.11_TX_D6")
 			(pintype "passive")
@@
 			(layers "*.Cu" "*.Mask")
 			(remove_unused_layers no)
-			(net 25 "Col 3")
+			(net 26 "Col 4")
 			(pinfunction "P1.11_TX_D6")
 			(pintype "passive")
@@
 		(fp_line
 			(start -0.35 0)
-			(end -0.35 0.550001)
+			(end -0.35 0.550002)
 			(stroke
 				(width 0.15)
@@
 		(fp_line
 			(start -1.4 -0.9)
-			(end -1.400001 0.900001)
+			(end -1.400002 0.900001)
 			(stroke
 				(width 0.1)
@@
 		)
 		(fp_line
-			(start 1.400001 -0.900001)
+			(start 1.400002 -0.900001)
 			(end -1.4 -0.9)
 			(stroke
@@
 		(fp_line
 			(start -0.35 0)
-			(end -0.35 0.550001)
+			(end -0.35 0.550002)
 			(stroke
 				(width 0.1)
@@
 		)
 		(fp_line
-			(start -1.400001 0.900001)
+			(start -1.400002 0.900001)
 			(end 1.4 0.9)
 			(stroke
@@
 		(fp_line
 			(start 1.4 0.9)
-			(end 1.400001 -0.900001)
+			(end 1.400002 -0.900001)
 			(stroke
 				(width 0.1)
@@
 	)
 	(segment
-		(start 124.522447 97.290641)
-		(end 129.694377 97.290641)
-		(width 0.2)
-		(layer "F.Cu")
-		(net 25)
-	)
-	(segment
 		(start 112.907011 59.078007)
 		(end 109.995415 61.989603)
@@
 	)
 	(segment
-		(start 141.995415 67.614603)
-		(end 143.920415 65.689603)
+		(start 109.995415 45.083066)
+		(end 109.995415 56.083077)
 		(width 0.2)
 		(layer "F.Cu")
@@
 	)
 	(segment
-		(start 109.995415 45.083066)
-		(end 109.995415 56.083077)
+		(start 112.988878 42.089603)
+		(end 109.995415 45.083066)
 		(width 0.2)
 		(layer "F.Cu")
@@
 	)
 	(segment
-		(start 141.995415 84.989603)
-		(end 141.995415 67.614603)
+		(start 143.155415 63.149603)
+		(end 144.755415 63.149603)
 		(width 0.2)
-		(layer "F.Cu")
+		(layer "B.Cu")
 		(net 25)
 	)
 	(segment
-		(start 129.694377 97.290641)
-		(end 141.995415 84.989603)
+		(start 134.829315 61.390603)
+		(end 141.396415 61.390603)
 		(width 0.2)
-		(layer "F.Cu")
+		(layer "B.Cu")
 		(net 25)
 	)
 	(segment
-		(start 112.988878 42.089603)
-		(end 109.995415 45.083066)
+		(start 141.396415 61.390603)
+		(end 143.155415 63.149603)
 		(width 0.2)
-		(layer "F.Cu")
+		(layer "B.Cu")
 		(net 25)
 	)
 	(segment
-		(start 130.990088 62.087695)
-		(end 142.858507 62.087695)
+		(start 112.990345 59.078007)
+		(end 132.516719 59.078007)
 		(width 0.2)
-		(layer "F.Cu")
-		(net 26)
+		(layer "B.Cu")
+		(net 25)
 	)
 	(segment
-		(start 145.182275 105.130053)
-		(end 142.396415 102.344193)
+		(start 132.516719 59.078007)
+		(end 134.829315 61.390603)
 		(width 0.2)
-		(layer "F.Cu")
-		(net 26)
+		(layer "B.Cu")
+		(net 25)
 	)
 	(segment
-		(start 142.858507 62.087695)
-		(end 143.920415 63.149603)
+		(start 127.995415 64.989603)
+		(end 127.995415 76.089603)
 		(width 0.2)
 		(layer "F.Cu")
@@
 	)
 	(segment
-		(start 127.995415 47.989603)
-		(end 127.995415 59.093022)
+		(start 127.995415 82.089603)
+		(end 127.995415 87.943193)
 		(width 0.2)
 		(layer "F.Cu")
@@
 	)
 	(segment
-		(start 142.396415 102.344193)
-		(end 142.396415 72.989603)
+		(start 127.995415 76.089603)
+		(end 130.995415 79.089603)
 		(width 0.2)
 		(layer "F.Cu")
@@
 	)
 	(segment
-		(start 142.396415 72.989603)
-		(end 146.995415 68.390603)
+		(start 133.995415 93.989603)
+		(end 134.041825 93.989603)
 		(width 0.2)
 		(layer "F.Cu")
@@
 	)
 	(segment
-		(start 128.077012 47.989603)
-		(end 127.995415 47.989603)
+		(start 130.995415 79.089603)
+		(end 127.995415 82.089603)
 		(width 0.2)
 		(layer "F.Cu")
@@
 	)
 	(segment
-		(start 127.995415 65.082368)
-		(end 127.995415 76.089603)
+		(start 144.395415 65.689603)
+		(end 144.755415 65.689603)
 		(width 0.2)
 		(layer "F.Cu")
@@
 	)
 	(segment
-		(start 146.995415 63.989603)
-		(end 146.155415 63.149603)
+		(start 127.995415 87.943193)
+		(end 145.182275 105.130053)
 		(width 0.2)
 		(layer "F.Cu")
@@
 	)
 	(segment
-		(start 127.995415 76.089603)
-		(end 130.995415 79.089603)
+		(start 130.897323 62.087695)
+		(end 127.995415 64.989603)
 		(width 0.2)
 		(layer "F.Cu")
@@
 	)
 	(segment
-		(start 130.990088 62.087695)
-		(end 127.995415 65.082368)
+		(start 127.995415 48.0712)
+		(end 127.995415 59.093022)
 		(width 0.2)
 		(layer "F.Cu")
@@
 	)
 	(segment
-		(start 146.995415 68.390603)
-		(end 146.995415 63.989603)
+		(start 130.984276 45.082339)
+		(end 127.995415 48.0712)
 		(width 0.2)
 		(layer "F.Cu")
@@
 	)
 	(segment
-		(start 130.984276 45.082339)
-		(end 128.077012 47.989603)
+		(start 130.995415 79.089603)
+		(end 144.395415 65.689603)
 		(width 0.2)
 		(layer "F.Cu")
@@
 	)
 	(segment
-		(start 146.155415 63.149603)
-		(end 144.755415 63.149603)
+		(start 130.990088 62.087695)
+		(end 130.897323 62.087695)
 		(width 0.2)
 		(layer "F.Cu")
@@
 	)
 	(zone
-		(net 0)
-		(net_name "")
+		(net 26)
+		(net_name "Col 4")
 		(layers "F.Cu" "B.Cu")
 		(hatch edge 0.5)
@@
 			(thermal_gap 0.5)
 			(thermal_bridge_width 0.5)
-			(island_removal_mode 1)
-			(island_area_min 10)
 		)
 		(polygon
 			(pts
-				(xy 45.995415 35.989603) (xy 87.995415 27.989603) (xy 171.995415 39.989603) (xy 155.995415 128.989603)
-				(xy 138.995415 127.989603) (xy 101.995415 111.989603) (xy 95.995415 98.989603) (xy 63.995415 109.989603)
-				(xy 40.995415 104.989603)
+				(xy 45.995415 28.989603) (xy 45.995415 110.989603) (xy 152.995415 132.989603) (xy 183.995415 30.989603)
 			)
 		)
