File: sweepish/sweepish.kicad_sch (KiCad schematic)
At the start: 35 parts, among them U1 XIAO-nRF52840-DIP

Commit message: Uploaded KiCad Files
Connections:
- net Col 3: now also U1.6 (P0.05_AIN3_A5_D5); no longer U1.7 (P1.11_TX_D6)
- net Col 4: now also U1.7 (P1.11_TX_D6); no longer U1.6 (P0.05_AIN3_A5_D5)
Changed lines of the file:
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@@
 	(global_label "Col 4"
 		(shape input)
-		(at 77.47 135.89 180)
+		(at 77.47 139.7 180)
 		(fields_autoplaced yes)
 		(effects
@@
 		)
 		(property "Intersheetrefs" "${INTERSHEET_REFS}"
-			(at 69.2235 135.89 0)
+			(at 69.2235 139.7 0)
 			(effects
 				(font
@@
 	(global_label "Col 3"
 		(shape input)
-		(at 77.47 139.7 180)
+		(at 77.47 135.89 180)
 		(fields_autoplaced yes)
 		(effects
@@
 		)
 		(property "Intersheetrefs" "${INTERSHEET_REFS}"
-			(at 69.2235 139.7 0)
+			(at 69.2235 135.89 0)
 			(effects
 				(font
